Commit message: tutorial prepared

File: urdf/robot40.urdf.xacro (robot description, xacro)
@@ -1,31 +1,12 @@
 <?xml version="1.0"?>
 <robot name="robot40" xmlns:xacro="http://ros.org/wiki/xacro">
-  <xacro:property name="headRadius" value="0.075" />
-  <xacro:property name="bodyLen" value="1.0" />
-  <xacro:property name="bodyRadius" value="0.075" />
-  <xacro:property name="shoulderLen" value="0.3" />
-  <xacro:property name="shoulderRadius" value="0.05" />
-  <xacro:property name="sideShoulderLen" value="0.15" />
-  <xacro:property name="sideShoulderRadius" value="0.05" />
   <xacro:property name="baseWidth" value="0.65" />
   <xacro:property name="baseLength" value="0.25" />
   <xacro:property name="baseHeight" value="0.15" />
+  <xacro:property name="baseMass" value="20" />
   <xacro:property name="wheeldiam" value="0.07" />
-  <xacro:property name="pi" value="3.1415" />
   <material name="blue">
     <color rgba="0 0 0.8 1"/>
   </material>
-  <material name="black">
-    <color rgba="0 0 0 1"/>
-  </material>
-  <material name="white">
-    <color rgba="1 1 1 1"/>
-  </material>
-  <xacro:macro name="default_inertial" params="mass">
-    <inertial>
-      <mass value="${mass}" />
-      <inertia ixx="1.0" ixy="0.0" ixz="0.0" iyy="1.0" iyz="0.0" izz="1.0" />
-    </inertial>
-  </xacro:macro>
   <link name="base_link">
     <visual>
@@ -40,7 +21,92 @@
       </geometry>
     </collision>
-    <xacro:default_inertial mass="40"/>
+    <inertial>
+      <mass value="${baseMass}" />
+      <inertia ixx="1.0" ixy="0.0" ixz="0.0" iyy="1.0" iyz="0.0" izz="1.0" />
+    </inertial>
   </link>
-<!--  <xacro:macro name="wheel" params="prefix suffix reflect">
+    <link name="body_link">
+    <visual>
+    <origin xyz="0.0 0.0 0.2" rpy="0 0 0" />
+        <geometry>
+        <mesh filename="package://urdf_example/meshes/robot40base.dae" />
+        </geometry>
+    </visual>
+    <collision>
+        <origin xyz="0.0 0.0 0.2" rpy="0 0 0" />
+        <geometry>
+          <mesh filename="package://urdf_example/meshes/robot40base.dae" />
+        </geometry>
+    </collision>
+    <inertial>
+        <mass value="10" />
+        <inertia ixx="1.0" ixy="0.0" ixz="0.0" iyy="1.0" iyz="0.0" izz="1.0" />
+    </inertial>
+    </link>
+  <joint name="base2body" type="fixed">
+    <axis xyz="0 1 0" rpy="0 0 0" />
+    <child link="body_link"/>
+    <parent link="base_link"/>
+    <origin xyz="0 0 0" rpy="0 0 0"/>
+  </joint>
+    <link name="head">
+      <visual>
+	<origin xyz="-0.14 0 1.323" rpy="0 0 -1.5708" />
+	<geometry>
+          <mesh filename="package://urdf_example/meshes/headBase.dae" />
+	</geometry>
+      </visual>
+      <collision>
+          <origin xyz="-0.14 0 1.323" rpy="0 0 -1.5708" />
+	<geometry>
+          <mesh filename="package://urdf_example/meshes/headBase.dae" />
+	</geometry>
+      </collision>
+      <inertial>
+        <mass value="2" />
+        <inertia ixx="1.0" ixy="0.0" ixz="0.0" iyy="1.0" iyz="0.0" izz="1.0" />
+    </inertial>
+    </link>
+    <joint name="toHead" type="fixed">
+        <parent link="body_link"/>
+        <child link="head"/>
+        <origin xyz="0 0 0"/>
+    </joint>
+    <link name="utm30">
+    <visual>
+        <origin xyz="0 0 0" rpy="1.5708 0 0.0" />
+        <geometry>
+        <mesh filename="package://urdf_example/meshes/headUTM.dae" />
+        </geometry>
+    </visual>
+    <collision>
+        <origin xyz="0 0 0" rpy="1.5708 0 0.0" />
+        <geometry>
+        <mesh filename="package://urdf_example/meshes/headUTM.dae" />
+        </geometry>
+    </collision>
+    <inertial>
+        <mass value="2" />
+        <inertia ixx="1.0" ixy="0.0" ixz="0.0" iyy="1.0" iyz="0.0" izz="1.0" />
+    </inertial>
+    </link>
+  <joint name="head_swivel" type="continuous">
+    <parent link="head"/>
+    <child link="utm30"/>
+    <axis xyz="0 1 0"/>
+    <origin xyz="-0.14 0.001 1.478" rpy="0 0 0"/>
+    <limit effort="30" velocity="1.0"/>
+    <dynamics damping="0.0" friction="0.0"/>
+  </joint>
+  <transmission name="head_swivel_trans">
+    <type>transmission_interface/SimpleTransmission</type>
+    <actuator name="$head_swivel_motor">
+      <mechanicalReduction>1</mechanicalReduction>
+    </actuator>
+    <joint name="head_swivel">
+      <hardwareInterface>PositionJointInterface</hardwareInterface>
+    </joint>
+  </transmission>
+  <xacro:macro name="wheel" params="prefix suffix reflect">
     <link name="${prefix}_${suffix}_wheel">
       <visual>
@@ -57,5 +123,8 @@
         </geometry>
       </collision>
-      <xacro:default_inertial mass="1"/>
+      <inertial>
+        <mass value="1" />
+        <inertia ixx="1.0" ixy="0.0" ixz="0.0" iyy="1.0" iyz="0.0" izz="1.0" />
+    </inertial>
     </link>
     <joint name="${prefix}_${suffix}_wheel_joint" type="continuous">
@@ -87,85 +156,13 @@
   </xacro:macro>
   <xacro:leg prefix="right" reflectLeg="-1" />
-  <xacro:leg prefix="left" reflectLeg="1" />-->
-<!--  <link name="body_link">
-      <visual>
-	<origin xyz="-0.00 -0.00 -0.45" rpy="0 0 0" />
-	<geometry>
-          <mesh filename="package://robot40sim/meshes/robot40base.dae" />
-	</geometry>
-      </visual>
-      <collision>
-          <origin xyz="-0.00 -0.0 -0.45" rpy="0 0 0" />
-	<geometry>
-          <mesh filename="package://robot40sim/meshes/robot40base.dae" />
-	</geometry>
-      </collision>
-      <xacro:cylinder_inertial radius="0.003" length="0.01" mass="${base_mass}">
-        <origin xyz="0.0 0.0 0.0" rpy="0 0 0" />
-      </xacro:cylinder_inertial>
-    </link>
-  <joint name="base2body" type="fixed">
-    <axis xyz="0 1 0" rpy="0 0 0" />
-    <child link="body_link"/>
-    <parent link="base_link"/>
-    <origin xyz="0 0 ${bodyLen/2+baseHeight/2}" rpy="0 0 0"/>
-  </joint>-->
-<!--    <link name="head">
-      <visual>
-	<origin xyz="-0.00 0.0 -0.0" rpy="0 0 -1.5708" />
-	<geometry>
-          <mesh filename="package://robot40sim/meshes/headBase.dae" />
-	</geometry>
-      </visual>
-      <collision>
-          <origin xyz="-0.00 0.0 -0.0" rpy="0 0 -1.5708" />
-	<geometry>
-          <mesh filename="package://robot40sim/meshes/headBase.dae" />
-	</geometry>
-      </collision>
-      <xacro:cylinder_inertial radius="0.003" length="0.005" mass="1.0">
-        <origin xyz="0.0 0.0 0.0" rpy="0 0 0" />
-      </xacro:cylinder_inertial>
-    </link>
-  <joint name="toHead" type="fixed">
-    <parent link="base_link"/>
-    <child link="head"/>
-    <origin xyz="-0.14 0 1.245"/>
-  </joint>-->
-<!--  <link name="utm30">
-    <visual>
-	<origin xyz="-0.00 0.0 -0.0" rpy="1.5708 0 0.0" />
-	<geometry>
-          <mesh filename="package://robot40sim/meshes/headUTM.dae" />
-	</geometry>
-      </visual>
-      <collision>
-          <origin xyz="-0.00 0.0 -0.0" rpy="0 0 0.0" />
-	<geometry>
-          <mesh filename="package://robot40sim/meshes/headUTM.dae" />
-	</geometry>
-      </collision>
-      <xacro:cylinder_inertial radius="0.003" length="0.005" mass="0.2">
-        <origin xyz="0.0 0.0 0.0" rpy="0 0 0" />
-      </xacro:cylinder_inertial>
-  </link>
-  <joint name="head_swivel" type="continuous">
-    <parent link="head"/>
-    <child link="utm30"/>
-    <axis xyz="0 0 1"/>
-    <origin xyz="0.0 0.001 0.155" rpy="0 0 0"/>
-    <limit effort="30" velocity="1.0"/>
-    <dynamics damping="0.0" friction="0.0"/>
+  <xacro:leg prefix="left" reflectLeg="1" />
+  <xacro:include filename="$(find ur_description)/urdf/ur3.urdf.xacro" />
+  <xacro:ur3_robot prefix="left_arm_" joint_limited="true"/>
+  <joint name="left_arm_shoulder" type="fixed">
+    <parent link="base_link" />
+    <child link = "left_arm_base_link" />
+    <origin xyz="-0.15 0.21 1.26" rpy="-2.3562 0.0 0.0" />
   </joint>
-  <transmission name="head_swivel_trans">
-    <type>transmission_interface/SimpleTransmission</type>
-    <actuator name="$head_swivel_motor">
-      <mechanicalReduction>1</mechanicalReduction>
-    </actuator>
-    <joint name="head_swivel">
-      <hardwareInterface>PositionJointInterface</hardwareInterface>
-    </joint>
-  </transmission>-->
-<!--  <gazebo reference="utm30">
+  <gazebo reference="utm30">
     <sensor type="camera" name="camera1">
       <update_rate>30.0</update_rate>
@@ -202,9 +199,9 @@
       </plugin>
     </sensor>
-  </gazebo>-->
-<!--    <gazebo reference="utm30">
+  </gazebo>
+  <gazebo reference="utm30">
         <sensor type="ray" name="head_hokuyo_sensor">
         <pose>0 0 0 0 0 0</pose>
-        <visualize>false</visualize>
+        <visualize>true</visualize>
         <update_rate>40</update_rate>
         <ray>
@@ -233,18 +230,5 @@
         </plugin>
         </sensor>
-    </gazebo>-->
-  <xacro:include filename="$(find ur_description)/urdf/ur3.urdf.xacro" />
-<!--   <xacro:ur3_robot prefix="left_arm_" joint_limited="true"/> -->
-<!--   <xacro:ur3_robot prefix="right_arm_" joint_limited="true"/> -->
-<!--  <joint name="left_arm_shoulder" type="fixed">
-    <parent link="base_link" />
-    <child link = "left_arm_base_link" />
-    <origin xyz="-0.15 0.21 1.19" rpy="-2.3562 0.0 0.0" />
-  </joint>-->
-  <!--<joint name="right_arm_shoulder" type="fixed">
-    <parent link="base_link" />
-    <child link = "right_arm_base_link" />
-    <origin xyz="-0.15 -0.21 1.19" rpy="2.3562 0.0 0.0" />
-  </joint>-->
+    </gazebo>
   <!-- Gazebo plugin for ROS Control -->
   <gazebo>
